Commit message: ros2 port

File: urdf/accessories.urdf.xacro (robot description, xacro)
@@ -2,6 +2,6 @@
 <robot xmlns:xacro="http://ros.org/wiki/xacro">
     <xacro:macro name="accessories" params="base_name base_length base_height  " >
-        <xacro:include filename="$(find hector_sensors_description)/urdf/hokuyo_utm30lx.urdf.xacro" />
-        <xacro:include filename="$(find hector_sensors_description)/urdf/asus_camera.urdf.xacro" />
+        <xacro:include filename="$(find mini_pupper_description)/urdf/hokuyo_utm30lx.urdf.xacro" />
+        <xacro:include filename="$(find mini_pupper_description)/urdf/asus_camera.urdf.xacro" />
         <xacro:hokuyo_utm30lx
             name="hokuyo"
@@ -12,5 +12,5 @@
             min_angle="130"
             max_angle="-130" >
-            <origin xyz="-0.05 0.0 ${base_height + 0.03}" rpy="0 0 0"/>
+            <origin xyz="0.0 0.0 ${base_height / 2 + 0.04}" rpy="0 0 0"/>
         </xacro:hokuyo_utm30lx>
         <xacro:asus_camera
@@ -19,17 +19,4 @@
             <origin xyz="${base_length / 2} 0.0 ${base_height + 0.012}" rpy="0 0 0"/>
         </xacro:asus_camera>
-        <gazebo>
-            <plugin name="imu_controller" filename="libhector_gazebo_ros_imu.so">
-                <updateRate>50.0</updateRate>
-                <bodyName>imu_link</bodyName>
-                <topicName>imu/data</topicName>
-                <accelDrift>0.005 0.005 0.005</accelDrift>
-                <accelGaussianNoise>0.005 0.005 0.005</accelGaussianNoise>
-                <rateDrift>0.005 0.005 0.005 </rateDrift>
-                <rateGaussianNoise>0.005 0.005 0.005 </rateGaussianNoise>
-                <headingDrift>0.005</headingDrift>
-                <headingGaussianNoise>0.005</headingGaussianNoise>
-            </plugin>
-        </gazebo>
         <link name="imu_link">
             <inertial>
@@ -43,4 +30,25 @@
             <child link="imu_link" />
         </joint>
+        <gazebo reference="imu_link">
+                <sensor name="imu_controller" type="imu">
+                    <always_on>true</always_on>
+                    <update_rate>50</update_rate>
+                    <plugin name="gazebo_ros_imu_sensor" filename="libgazebo_ros_imu_sensor.so">
+                        <ros>
+                            <namespace>/imu</namespace>
+                            <argument>~/out:=data</argument>
+                        </ros>
+                        <!-- <updateRate>50.0</updateRate>
+                        <bodyName>imu_link</bodyName>
+                        <topicName>imu/data</topicName>
+                        <accelDrift>0.005 0.005 0.005</accelDrift>
+                        <accelGaussianNoise>0.005 0.005 0.005</accelGaussianNoise>
+                        <rateDrift>0.005 0.005 0.005 </rateDrift>
+                        <rateGaussianNoise>0.005 0.005 0.005 </rateGaussianNoise>
+                        <headingDrift>0.005</headingDrift>
+                        <headingGaussianNoise>0.005</headingGaussianNoise> -->
+                    </plugin>
+                </sensor>
+            </gazebo>
         <!-- <xacro:include filename="$(find velodyne_description)/urdf/VLP-16.urdf.xacro"/>
         <xacro:VLP-16 parent="${base_name}" name="velodyne" topic="velodyne_points" hz="10" samples="1024" gpu="false" lasers="16" max_range="100">

File: urdf/accessories_another.urdf.xacro (robot description, xacro)
@@ -2,14 +2,14 @@
 <robot xmlns:xacro="http://ros.org/wiki/xacro">
     <xacro:macro name="accessories" params="base_name base_length base_height  " >
-        <xacro:include filename="$(find mini-pupper_description)/urdf/ld06.urdf.xacro" />
+        <xacro:include filename="$(find mini_pupper_description)/urdf/ld06.urdf.xacro" />
         <xacro:include filename="$(find realsense2_description)/urdf/_d435i.urdf.xacro" />
         <xacro:ld06
             parent="${base_name}" >
-            <origin xyz="-0.05 0.0 ${base_height / 2 + 0.060}" rpy="0 0 0"/>
+            <origin xyz="-0.05 0.0 ${base_height / 2 + 0.030}" rpy="0 0 0"/>
         </xacro:ld06>
         <xacro:sensor_d435i
             parent="${base_name}"
             name="camera">
-            <origin xyz="${base_length / 2 + 0.01} 0.0 ${base_height - 0.025}" rpy="0 0 0"/>
+            <origin xyz="${base_length / 2} 0.0 ${base_height + 0.012}" rpy="0 0 0"/>
         </xacro:sensor_d435i>
         <gazebo>

File: urdf/ld06.urdf.xacro (robot description, xacro)
@@ -2,5 +2,5 @@
 <robot xmlns:xacro="http://ros.org/wiki/xacro">
   <xacro:macro name="ld06" params="*origin parent">
-    <xacro:include filename="$(find mini-pupper_description)/urdf/laser.urdf.xacro" />
+    <xacro:include filename="$(find mini_pupper_description)/urdf/laser.urdf.xacro" />
     <xacro:laser
       parent="${parent}"

File: urdf/leg.urdf.xacro (robot description, xacro)
@@ -6,7 +6,7 @@
             <xacro:property name="hip_to_upper_leg" value="${hip_to_upper_leg_distance}" />
             <xacro:property name="upper_leg_to_lower_leg" value="${upper_leg_to_lower_leg_distance}" />
-            <xacro:property name="hip_mesh_path" value="package://mini-pupper_description/meshes/${leg}_hip.stl" />
-            <xacro:property name="upper_leg_mesh_path" value="package://mini-pupper_description/meshes/${leg}_lower_leg.stl" />
-            <xacro:property name="lower_leg_mesh_path" value="package://mini-pupper_description/meshes/${leg}_lower_leg.stl" />
+            <xacro:property name="hip_mesh_path" value="file://$(find mini_pupper_description)/meshes/${leg}_hip.stl" />
+            <xacro:property name="upper_leg_mesh_path" value="file://$(find mini_pupper_description)/meshes/${leg}_lower_leg.stl" />
+            <xacro:property name="lower_leg_mesh_path" value="file://$(find mini_pupper_description)/meshes/${leg}_lower_leg.stl" />
         </xacro:if>
         <xacro:if value="${leg == 'lh'}">
@@ -14,7 +14,7 @@
             <xacro:property name="hip_to_upper_leg" value="${hip_to_upper_leg_distance}" />
             <xacro:property name="upper_leg_to_lower_leg" value="${upper_leg_to_lower_leg_distance}" />
-            <xacro:property name="hip_mesh_path" value="package://mini-pupper_description/meshes/${leg}_hip.stl" />
-            <xacro:property name="upper_leg_mesh_path" value="package://mini-pupper_description/meshes/${leg}_lower_leg.stl" />
-            <xacro:property name="lower_leg_mesh_path" value="package://mini-pupper_description/meshes/${leg}_lower_leg.stl" />
+            <xacro:property name="hip_mesh_path" value="file://$(find mini_pupper_description)/meshes/${leg}_hip.stl" />
+            <xacro:property name="upper_leg_mesh_path" value="file://$(find mini_pupper_description)/meshes/${leg}_lower_leg.stl" />
+            <xacro:property name="lower_leg_mesh_path" value="file://$(find mini_pupper_description)/meshes/${leg}_lower_leg.stl" />
         </xacro:if>
         <xacro:if value="${leg == 'rf'}">
@@ -22,7 +22,7 @@
             <xacro:property name="hip_to_upper_leg" value="-${hip_to_upper_leg_distance}" />
             <xacro:property name="upper_leg_to_lower_leg" value="-${upper_leg_to_lower_leg_distance}" />
-            <xacro:property name="hip_mesh_path" value="package://mini-pupper_description/meshes/${leg}_hip.stl" />
-            <xacro:property name="upper_leg_mesh_path" value="package://mini-pupper_description/meshes/${leg}_lower_leg.stl" />
-            <xacro:property name="lower_leg_mesh_path" value="package://mini-pupper_description/meshes/${leg}_lower_leg.stl" />
+            <xacro:property name="hip_mesh_path" value="file://$(find mini_pupper_description)/meshes/${leg}_hip.stl" />
+            <xacro:property name="upper_leg_mesh_path" value="file://$(find mini_pupper_description)/meshes/${leg}_lower_leg.stl" />
+            <xacro:property name="lower_leg_mesh_path" value="file://$(find mini_pupper_description)/meshes/${leg}_lower_leg.stl" />
         </xacro:if>
         <xacro:if value="${leg == 'rh'}">
@@ -30,7 +30,7 @@
             <xacro:property name="hip_to_upper_leg" value="-${hip_to_upper_leg_distance}" />
             <xacro:property name="upper_leg_to_lower_leg" value="-${upper_leg_to_lower_leg_distance}" />
-            <xacro:property name="hip_mesh_path" value="package://mini-pupper_description/meshes/${leg}_hip.stl" />
-            <xacro:property name="upper_leg_mesh_path" value="package://mini-pupper_description/meshes/${leg}_lower_leg.stl" />
-            <xacro:property name="lower_leg_mesh_path" value="package://mini-pupper_description/meshes/${leg}_lower_leg.stl" />
+            <xacro:property name="hip_mesh_path" value="file://$(find mini_pupper_description)/meshes/${leg}_hip.stl" />
+            <xacro:property name="upper_leg_mesh_path" value="file://$(find mini_pupper_description)/meshes/${leg}_lower_leg.stl" />
+            <xacro:property name="lower_leg_mesh_path" value="file://$(find mini_pupper_description)/meshes/${leg}_lower_leg.stl" />
         </xacro:if>
         <link name="${leg}_hip_debug_link"/>
@@ -107,6 +107,6 @@
         </link>
         <gazebo reference="${leg}_lower_leg_link">
-            <kp>1000000.0</kp>
-            <kd>1.0</kd>
+            <kp>10000000000.0</kp>
+            <kd>100.0</kd>
             <mu1>0.8</mu1>
             <mu2>0.8</mu2>
@@ -201,4 +201,24 @@
             </actuator>
         </transmission>
+        <ros2_control name="${leg}" type="system">
+            <hardware>
+                <plugin>gazebo_ros2_control/GazeboSystem</plugin>
+            </hardware>
+            <joint name="${leg}_hip_joint">
+                <command_interface name="effort"/>
+                <state_interface name="position"/>
+                <state_interface name="velocity"/>
+            </joint>
+            <joint name="${leg}_upper_leg_joint">
+                <command_interface name="effort"/>
+                <state_interface name="position"/>
+                <state_interface name="velocity"/>
+            </joint>
+            <joint name="${leg}_lower_leg_joint">
+                <command_interface name="effort"/>
+                <state_interface name="position"/>
+                <state_interface name="velocity"/>
+            </joint>
+        </ros2_control>
     </xacro:macro>
 </robot>

File: urdf/mini-pupper.urdf.xacro (robot description, xacro)
@@ -1,5 +1,5 @@
 <?xml version="1.0"?>
 <robot name="mini-pupper" xmlns:xacro="http://ros.org/wiki/xacro">
-    <xacro:include filename="$(find mini-pupper_description)/urdf/properties.urdf.xacro" />
+    <xacro:include filename="$(find mini_pupper_description)/urdf/properties.urdf.xacro" />
     <material name="black"><color rgba="0.15 0.15 0.15 1.0" /></material>
     <material name="dyellow"><color rgba="0.95 0.93 0.13 1.0" /></material>
@@ -15,5 +15,5 @@
             <origin xyz="0 0 0" rpy="0 0 0" />
             <geometry>
-                <mesh filename="package://mini-pupper_description/meshes/base.stl" scale="1 1 1" />
+                <mesh filename="file://$(find mini_pupper_description)/meshes/base.stl" scale="1 1 1" />
             </geometry>
             <material name="dyellow" />
@@ -104,6 +104,6 @@
         <material>Gazebo/White</material>
     </gazebo> -->
-    <xacro:include filename="$(find mini-pupper_description)/urdf/leg.urdf.xacro" />
-    <xacro:include filename="$(find mini-pupper_description)/urdf/accessories.urdf.xacro" />
+    <xacro:include filename="$(find mini_pupper_description)/urdf/leg.urdf.xacro" />
+    <xacro:include filename="$(find mini_pupper_description)/urdf/accessories.urdf.xacro" />
     <xacro:accessories
         base_name="base_link"
@@ -128,7 +128,7 @@
     </gazebo>
     <gazebo>
-        <plugin name="gazebo_ros_control" filename="libgazebo_ros_control.so">
-            <legacyModeNS>true</legacyModeNS>
-        </plugin>
+        <plugin filename="libgazebo_ros2_control.so" name="gazebo_ros2_control">
+        <parameters>$(find mini_pupper_description)/config/ros_control.yaml</parameters>
+      </plugin>
     </gazebo>
 </robot>

File: urdf/mini_pupper.urdf (robot description, URDF)
Before this commit: robot mini-pupper, 29 links, 28 joints
Links:
- link base_link: geometry collision mesh filename=file:///home/juan/champ2_ws/install/mini_pupper_description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 scale=0.001 0.001 0.001; visual mesh filename=file:///home/juan/champ2_ws/install/mini_pupper_description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 scale=1 1 1
- link camera_link: geometry collision mesh filename=file:///home/juan/champ2_ws/install/champ_description/share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; visual mesh filename=file:///home/juan/champ2_ws/install/champ_description/share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
- link hokuyo_frame: geometry collision box size=0.058 0.058 0.087; visual mesh filename=file:///home/juan/champ2_ws/install/champ_description/share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
- link lf_foot_link: geometry collision mesh filename=file:///home/juan/champ2_ws/install/mini_pupper_description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 scale=1 1 1; visual mesh filename=file:///home/juan/champ2_ws/install/mini_pupper_description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 scale=1 1 1
- link lf_hip_link: geometry collision mesh filename=file:///home/juan/champ2_ws/install/mini_pupper_description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 scale=1 1 1; visual mesh filename=file:///home/juan/champ2_ws/install/mini_pupper_description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 scale=1 1 1
- link lf_lower_leg_link: geometry collision mesh filename=file:///home/juan/champ2_ws/install/mini_pupper_description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 scale=1 1 1; visual mesh filename=file:///home/juan/champ2_ws/install/mini_pupper_description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 scale=1 1 1
- link lf_upper_leg_link: geometry collision mesh filename=file:///home/juan/champ2_ws/install/mini_pupper_description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 scale=1 1 1; visual mesh filename=file:///home/juan/champ2_ws/install/mini_pupper_description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 scale=1 1 1
- link lh_foot_link: geometry collision mesh filename=file:///home/juan/champ2_ws/install/mini_pupper_description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 scale=1 1 1; visual mesh filename=file:///home/juan/champ2_ws/install/mini_pupper_description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 scale=1 1 1
- link lh_hip_link: geometry collision mesh filename=file:///home/juan/champ2_ws/install/mini_pupper_description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 scale=1 1 1; visual mesh filename=file:///home/juan/champ2_ws/install/mini_pupper_description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 scale=1 1 1
- link lh_lower_leg_link: geometry collision mesh filename=file:///home/juan/champ2_ws/install/mini_pupper_description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 scale=1 1 1; visual mesh filename=file:///home/juan/champ2_ws/install/mini_pupper_description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 scale=1 1 1
- link lh_upper_leg_link: geometry collision mesh filename=file:///home/juan/champ2_ws/install/mini_pupper_description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 scale=1 1 1; visual mesh filename=file:///home/juan/champ2_ws/install/mini_pupper_description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 scale=1 1 1
- link rf_foot_link: geometry collision mesh filename=file:///home/juan/champ2_ws/install/mini_pupper_description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 scale=1 1 1; visual mesh filename=file:///home/juan/champ2_ws/install/mini_pupper_description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 scale=1 1 1
- link rf_hip_link: geometry collision mesh filename=file:///home/juan/champ2_ws/install/mini_pupper_description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 scale=1 1 1; visual mesh filename=file:///home/juan/champ2_ws/install/mini_pupper_description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 scale=1 1 1
- link rf_lower_leg_link: geometry collision mesh filename=file:///home/juan/champ2_ws/install/mini_pupper_description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 scale=1 1 1; visual mesh filename=file:///home/juan/champ2_ws/install/mini_pupper_description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 scale=1 1 1
- link rf_upper_leg_link: geometry collision mesh filename=file:///home/juan/champ2_ws/install/mini_pupper_description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 scale=1 1 1; visual mesh filename=file:///home/juan/champ2_ws/install/mini_pupper_description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 scale=1 1 1
- link rh_foot_link: geometry collision mesh filename=file:///home/juan/champ2_ws/install/mini_pupper_description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 scale=1 1 1; visual mesh filename=file:///home/juan/champ2_ws/install/mini_pupper_description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 scale=1 1 1
- link rh_hip_link: geometry collision mesh filename=file:///home/juan/champ2_ws/install/mini_pupper_description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 scale=1 1 1; visual mesh filename=file:///home/juan/champ2_ws/install/mini_pupper_description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 scale=1 1 1
- link rh_lower_leg_link: geometry collision mesh filename=file:///home/juan/champ2_ws/install/mini_pupper_description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 scale=1 1 1; visual mesh filename=file:///home/juan/champ2_ws/install/mini_pupper_description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 scale=1 1 1
- link rh_upper_leg_link: geometry collision mesh filename=file:///home/juan/champ2_ws/install/mini_pupper_description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 scale=1 1 1; visual mesh filename=file:///home/juan/champ2_ws/install/mini_pupper_description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 scale=1 1 1
Joints:
- joint camera_joint: origin xyz=0.098 0.0 0.082 rpy=0 0 0 -> xyz=0.098 0.0 -0.045000000000000005 rpy=0 0 0
- joint hokuyo_joint: origin xyz=-0.05 0.0 0.1 rpy=0 0 0 -> xyz=0.0 0.0 0.07500000000000001 rpy=0 0 0

File: urdf/properties.urdf.xacro (robot description, xacro)
@@ -20,5 +20,5 @@
     <xacro:property name="lower_leg_y_length" value="0.0015" />
     <xacro:property name="lower_leg_z_length" value="0.07844" />
-    <xacro:property name="base_mesh_path" value="package://mini-pupper_description/meshes/base.stl" />
+    <xacro:property name="base_mesh_path" value="file://$(find mini_pupper_description)/meshes/base.stl" />
     <xacro:property name="base_mass" value="1.0" />
     <!-- <xacro:property name="base_mass" value="2.0" /> -->
@@ -26,5 +26,5 @@
     <xacro:property name="base_y_length" value="0.07" />
     <xacro:property name="base_z_length" value="0.07" />
-    <xacro:property name="foot_mesh_path" value="package://mini-pupper_description/meshes/foot.stl" />
+    <xacro:property name="foot_mesh_path" value="file://$(find mini_pupper_description)/meshes/foot.stl" />
     <xacro:property name="foot_mass" value="0.0625" />
     <xacro:property name="foot_x_length" value="0.017" />
